File: Didaktik multilayout.kicad_pcb (KiCad board)
At the start: 2 copper layers, 209.6 x 76.2 mm, 130 parts, among them J1 Conn_01x04_MountingPin, J2 AVR-ISP-6, SW1 SW_Push_45deg, SW10 SW_Push_45deg, SW11 SW_Push_45deg, SW12 SW_Push_45deg, SW13 SW_Push_45deg, SW14 SW_Push_45deg, SW15 SW_Push_45deg, SW16 SW_Push_45deg, SW17 SW_Push_45deg, SW18 SW_Push_45deg, SW19 SW_Push_45deg, SW2 SW_Push_45deg, SW20 SW_Push_45deg, SW21 SW_Push_45deg, SW22 SW_Push_45deg, SW23 SW_Push_45deg, SW24 SW_Push_45deg, SW25 SW_Push_45deg, SW26 SW_Push_45deg, SW27 SW_Push_45deg, SW28 SW_Push_45deg, SW29 SW_Push_45deg, SW3 SW_Push_45deg, SW30 SW_Push_45deg, SW31 SW_Push_45deg, SW31a1 SW_Push_45deg, SW32 SW_Push_45deg, SW32a1 SW_Push_45deg, SW33 SW_Push_45deg, SW33a1 SW_Push_45deg, SW34 SW_Push_45deg, SW34a1 SW_Push_45deg, SW34b1 SW_Push_45deg, SW35 SW_Push_45deg, SW35a1 SW_Push_45deg, SW35b1 SW_Push_45deg, SW35c1 SW_Push_45deg, SW36 SW_Push_45deg, SW36a1 SW_Push_45deg, SW36b1 SW_Push_45deg, SW36c1 SW_Push_45deg, SW37 SW_Push_45deg, SW37a1 SW_Push_45deg, SW37b1 SW_Push_45deg, SW38 SW_Push_45deg, SW38a1 SW_Push_45deg, SW39 SW_Push_45deg, SW39a1 SW_Push_45deg, SW4 SW_Push_45deg, SW40 SW_Push_45deg, SW40a1 SW_Push_45deg, SW5 SW_Push_45deg, SW6 SW_Push_45deg, SW7 SW_Push_45deg, SW8 SW_Push_45deg, SW9 SW_Push_45deg, U1 ATmega32U4-M, Y1 Crystal_GND24_Small

Commit message: cleaning up pcb & switch plate edge cut
Other:
- board text added: "case dimensions"
- board text added: "hole alignment and size?"
- board text added: "move jst connector down?"
- board text added: "plate, pcb edge to case edge, overlap?"
Changed lines of the file:
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@@
     (property "Sheetname" "")
     (attr smd)
-    (fp_text reference "F1" (at 0 1.82 90) (layer "B.SilkS")
+    (fp_text reference "F1" (at 0 1.82 90) (layer "B.SilkS") hide
       (effects (font (size 1 1) (thickness 0.15)) (justify mirror))
     )
@@
     (property "Sheetname" "")
     (attr through_hole)
-    (fp_text reference "J1" (at 0 6.5) (layer "B.SilkS")
+    (fp_text reference "J1" (at 0 6.5) (layer "B.SilkS") hide
       (effects (font (size 1 1) (thickness 0.15)) (justify mirror))
     )
@@
     (property "Sheetname" "")
     (attr smd)
-    (fp_text reference "D25" (at 0.02 2.38) (layer "B.SilkS")
+    (fp_text reference "D25" (at 0.02 2.38) (layer "B.SilkS") hide
       (effects (font (size 1 1) (thickness 0.15)) (justify mirror))
     )
@@
   )
   (gr_rect (start 3.175 -25.4) (end 269.875 136.525) (layer "B.Cu") (width 0.15) (fill none))
-  (gr_line (start 31.75 107.95) (end 12.7 107.95) (layer "Cmts.User") (width 0.2))
-  (gr_line (start 241.3 107.95) (end 260.35 107.95) (layer "Cmts.User") (width 0.15))
+  (gr_circle (center 236.5375 46.0375) (end 238.782564 46.0375) (layer "Cmts.User") (width 0.1) (fill none))
+  (gr_line (start 31.75 88.9) (end 12.7 88.9) (layer "Cmts.User") (width 0.2))
+  (gr_line (start 33.3375 107.95) (end 239.7125 107.95) (layer "Cmts.User") (width 0.2))
+  (gr_line (start 222.25 31.75) (end 222.25 50.8) (layer "Cmts.User") (width 0.2))
+  (gr_line (start 31.75 50.8) (end 41.275 50.8) (layer "Cmts.User") (width 0.2))
+  (gr_line (start 239.7125 107.95) (end 260.35 107.95) (layer "Cmts.User") (width 0.2))
   (gr_rect (start 12.7 -6.35) (end 260.35 127) (layer "Cmts.User") (width 0.2) (fill none))
+  (gr_arc (start 241.3 106.3625) (mid 240.835032 107.485032) (end 239.7125 107.95) (layer "Cmts.User") (width 0.2))
   (gr_line (start 12.7 17.4625) (end 260.35 17.4625) (layer "Cmts.User") (width 0.15))
   (gr_line (start 165.1 17.4625) (end 169.8625 3.175) (layer "Cmts.User") (width 0.15))
+  (gr_line (start 50.8 69.85) (end 41.275 69.85) (layer "Cmts.User") (width 0.2))
+  (gr_line (start 41.275 69.85) (end 12.7 69.85) (layer "Cmts.User") (width 0.15))
+  (gr_line (start 33.3375 107.95) (end 12.7 107.95) (layer "Cmts.User") (width 0.2))
   (gr_line (start 31.75 50.8) (end 12.7 50.8) (layer "Cmts.User") (width 0.2))
+  (gr_arc (start 31.75 33.3375) (mid 32.214968 32.214968) (end 33.3375 31.75) (layer "Cmts.User") (width 0.2))
+  (gr_line (start 231.775 50.927) (end 231.775 69.85) (layer "Cmts.User") (width 0.2))
   (gr_line (start 231.775 50.8) (end 260.35 50.8) (layer "Cmts.User") (width 0.15))
-  (gr_line (start 241.3 88.9) (end 260.35 88.9) (layer "Cmts.User") (width 0.15))
-  (gr_line (start 222.25 31.75) (end 260.35 31.75) (layer "Cmts.User") (width 0.15))
+  (gr_line (start 231.775 69.85) (end 241.3 69.85) (layer "Cmts.User") (width 0.2))
+  (gr_line (start 41.275 69.85) (end 41.275 50.8) (layer "Cmts.User") (width 0.2))
+  (gr_line (start 241.3 88.9) (end 260.35 88.9) (layer "Cmts.User") (width 0.2))
+  (gr_line (start 50.8 88.9) (end 50.8 69.85) (layer "Cmts.User") (width 0.2))
+  (gr_line (start 222.25 31.75) (end 260.35 31.75) (layer "Cmts.User") (width 0.2))
   (gr_line (start 163.5125 17.4625) (end 168.275 3.175) (layer "Cmts.User") (width 0.15))
+  (gr_line (start 31.75 88.9) (end 50.8 88.9) (layer "Cmts.User") (width 0.2))
+  (gr_arc (start 33.3375 107.95) (mid 32.214968 107.485032) (end 31.75 106.3625) (layer "Cmts.User") (width 0.2))
   (gr_line (start 174.625 17.4625) (end 179.3875 3.175) (layer "Cmts.User") (width 0.15))
-  (gr_line (start 41.275 69.85) (end 12.7 69.85) (layer "Cmts.User") (width 0.2))
   (gr_line (start 12.7 3.175) (end 260.35 3.175) (layer "Cmts.User") (width 0.15))
-  (gr_line (start 31.75 88.9) (end 12.7 88.9) (layer "Cmts.User") (width 0.2))
+  (gr_line (start 31.75 33.3375) (end 31.75 50.8) (layer "Cmts.User") (width 0.2))
   (gr_line (start 171.45 17.4625) (end 176.2125 3.175) (layer "Cmts.User") (width 0.15))
+  (gr_line (start 241.3 69.85) (end 241.3 106.3625) (layer "Cmts.User") (width 0.2))
+  (gr_circle (center 236.5375 55.5625) (end 238.782564 55.5625) (layer "Cmts.User") (width 0.1) (fill none))
+  (gr_line (start 31.75 31.75) (end 222.25 31.75) (layer "Cmts.User") (width 0.2))
   (gr_line (start 190.5 17.4625) (end 195.2625 3.175) (layer "Cmts.User") (width 0.15))
   (gr_line (start 184.15 17.4625) (end 188.9125 3.175) (layer "Cmts.User") (width 0.15))
   (gr_line (start 31.75 31.75) (end 12.7 31.75) (layer "Cmts.User") (width 0.2))
+  (gr_line (start 222.25 50.8) (end 231.775 50.8) (layer "Cmts.User") (width 0.2))
+  (gr_line (start 31.75 88.9) (end 31.75 106.3625) (layer "Cmts.User") (width 0.2))
+  (gr_circle (center 236.560064 38.989) (end 238.805128 38.989) (layer "Cmts.User") (width 0.1) (fill none))
   (gr_line (start 179.3875 17.4625) (end 184.15 3.175) (layer "Cmts.User") (width 0.15))
-  (gr_line (start 241.3 69.85) (end 260.35 69.85) (layer "Cmts.User") (width 0.15))
+  (gr_line (start 241.3 69.85) (end 260.35 69.85) (layer "Cmts.User") (width 0.2))
   (gr_line (start 168.275 17.4625) (end 173.0375 3.175) (layer "Cmts.User") (width 0.15))
-  (gr_arc (start 33.3375 108.077) (mid 32.214968 107.612032) (end 31.75 106.4895) (layer "Edge.Cuts") (width 0.15))
-  (gr_line (start 33.3375 31.877) (end 239.7125 31.877) (layer "Edge.Cuts") (width 0.15))
-  (gr_line (start 31.75 106.4895) (end 31.75 33.4645) (layer "Edge.Cuts") (width 0.15))
-  (gr_arc (start 241.3 106.4895) (mid 240.835032 107.612032) (end 239.7125 108.077) (layer "Edge.Cuts") (width 0.15))
-  (gr_line (start 239.7125 108.077) (end 33.3375 108.077) (layer "Edge.Cuts") (width 0.15))
-  (gr_arc (start 239.7125 31.877) (mid 240.835032 32.341968) (end 241.3 33.4645) (layer "Edge.Cuts") (width 0.15))
-  (gr_arc (start 31.75 33.4645) (mid 32.214968 32.341968) (end 33.3375 31.877) (layer "Edge.Cuts") (width 0.15))
-  (gr_line (start 241.3 33.4645) (end 241.3 106.4895) (layer "Edge.Cuts") (width 0.15))
+  (gr_arc (start 33.3375 107.95) (mid 32.214968 107.485032) (end 31.75 106.3625) (layer "Edge.Cuts") (width 0.15))
+  (gr_line (start 33.3375 31.75) (end 239.7125 31.75) (layer "Edge.Cuts") (width 0.15))
+  (gr_line (start 31.75 106.3625) (end 31.75 33.3375) (layer "Edge.Cuts") (width 0.15))
+  (gr_arc (start 241.3 106.3625) (mid 240.835032 107.485032) (end 239.7125 107.95) (layer "Edge.Cuts") (width 0.15))
+  (gr_line (start 239.7125 107.95) (end 33.3375 107.95) (layer "Edge.Cuts") (width 0.15))
+  (gr_arc (start 239.7125 31.75) (mid 240.835032 32.214968) (end 241.3 33.3375) (layer "Edge.Cuts") (width 0.15))
+  (gr_arc (start 31.75 33.3375) (mid 32.214968 32.214968) (end 33.3375 31.75) (layer "Edge.Cuts") (width 0.15))
+  (gr_line (start 241.3 33.3375) (end 241.3 106.3625) (layer "Edge.Cuts") (width 0.15))
+  (gr_text "plate, pcb edge to case edge, overlap?" (at 8.001 55.118) (layer "F.Cu")
+    (effects (font (size 1.5 1.5) (thickness 0.3)))
+  )
+  (gr_text "case dimensions\n" (at 23.241 27.051) (layer "F.Cu")
+    (effects (font (size 1.5 1.5) (thickness 0.3)))
+  )
+  (gr_text "hole alignment and size?\n" (at 257.81 41.148) (layer "F.Cu")
+    (effects (font (size 1.5 1.5) (thickness 0.3)))
+  )
+  (gr_text "move jst connector down?\n" (at 236.855 29.591) (layer "F.Cu")
+    (effects (font (size 1.5 1.5) (thickness 0.3)))
+  )
   (gr_text "6U" (at 88.9 85.725) (layer "B.SilkS")
     (effects (font (size 1 1) (thickness 0.15)) (justify mirror))
@@
     (effects (font (size 1 1) (thickness 0.15)) (justify mirror))
   )
-  (gr_text "Didaktik 40 v1.0 by Calvin#0563" (at 61.595 33.528) (layer "B.SilkS")
-    (effects (font (size 2 2) (thickness 0.15)) (justify mirror))
+  (gr_text "Didaktik 40 v1.0 by Calvin#0563" (at 55.5625 33.528) (layer "B.SilkS")
+    (effects (font (size 1.75 1.75) (thickness 0.15)) (justify mirror))
   )
   (gr_text "6U" (at 184.15 85.725) (layer "B.SilkS")
@@
     (style (thickness 0.15) (arrow_length 1.27) (text_position_mode 0) (extension_height 0.58642) (extension_offset 0.5) keep_text_aligned)
   )
-  (dimension (type aligned) (layer "Cmts.User")
+  (dimension (type aligned) (layer "Dwgs.User")
     (pts (xy 11.40887 31.75) (xy 11.40887 108.103871))
     (height 32.04637)
-    (gr_text "76.3539 mm" (at -21.7875 69.926935 90) (layer "Cmts.User")
+    (gr_text "76.3539 mm" (at -21.7875 69.926935 90) (layer "Dwgs.User")
       (effects (font (size 1 1) (thickness 0.15)))
     )
@@
     (style (thickness 0.15) (arrow_length 1.27) (text_position_mode 0) (extension_height 0.58642) (extension_offset 0.5) keep_text_aligned)
   )
-  (dimension (type aligned) (layer "Cmts.User")
+  (dimension (type aligned) (layer "Dwgs.User")
     (pts (xy 260.35 127) (xy 260.35 -6.35))
     (height 12.7)
-    (gr_text "133.3500 mm" (at 271.25 60.325 90) (layer "Cmts.User")
+    (gr_text "133.3500 mm" (at 271.25 60.325 90) (layer "Dwgs.User")
       (effects (font (size 1.5 1.5) (thickness 0.3)))
     )
@@
     (style (thickness 0.2) (arrow_length 1.27) (text_position_mode 0) (extension_height 0.58642) (extension_offset 0.5) keep_text_aligned)
   )
-  (dimension (type aligned) (layer "Cmts.User")
+  (dimension (type aligned) (layer "Dwgs.User")
     (pts (xy 12.7 127) (xy 260.35 127))
     (height 6.35)
-    (gr_text "247.6500 mm" (at 136.525 131.55) (layer "Cmts.User")
+    (gr_text "247.6500 mm" (at 136.525 131.55) (layer "Dwgs.User")
       (effects (font (size 1.5 1.5) (thickness 0.3)))
     )
@@
     (style (thickness 0.2) (arrow_length 1.27) (text_position_mode 0) (extension_height 0.58642) (extension_offset 0.5) keep_text_aligned)
   )
-  (dimension (type aligned) (layer "Cmts.User")
+  (dimension (type aligned) (layer "Dwgs.User")
     (pts (xy 31.679333 129.634738) (xy 241.37312 129.634738))
     (height 10.065262)
-    (gr_text "209.6938 mm" (at 136.526226 138.55) (layer "Cmts.User")
+    (gr_text "209.6938 mm" (at 136.526226 138.55) (layer "Dwgs.User")
       (effects (font (size 1 1) (thickness 0.15)))
     )

Commit message: redoing JST placement, some routing, full  boardGND fill
Parts:
- moved F1 5.48 mm to (233.8, 48.8)
- moved D25 5.47 mm to (230.5, 46.1)
- moved J1 4.15 mm to (225.9, 38.1), turned to 90 degrees
- moved D42 1.59 mm to (236.5, 44.5)
- moved R8 1.59 mm to (239.7, 44.5)
- moved D43 0.91 mm to (236.5, 38.1)
- moved R9 0.90 mm to (239.8, 38.1)
Routing:
- net D+: track 226.8 -> 236.5 mm
- net (no net): track 8.71 -> 0.00 mm, vias 2 -> 0
- net D-: track 227.9 -> 236.2 mm
- net SCK: track 62.7 -> 55.6 mm, vias 3 -> 2
- net GND: track 90.8 -> 83.9 mm, vias 13 -> 12
- net VCC: track 15.9 -> 22.6 mm
- net MOSI: track 66.8 -> 60.6 mm, vias 3 -> 2
- net MISO: track 64.6 -> 59.2 mm, vias 3 -> 2
- net ROW0: track 418.2 -> 416.4 mm
- net LED Power: track 218.3 -> 219.9 mm
- net LED capslock: track 224.6 -> 225.5 mm
- net +5V: track 300.1 -> 300.8 mm
- net RESET: track 225.8 -> 226.3 mm, vias 1 -> 3
Other:
- board text removed: "hole alignment and size?"
- board text removed: "move jst connector down?"
- board text removed: "plate, pcb edge to case edge, overlap?"
