File: Didaktik switchplate.kicad_pcb (KiCad board)
At the start: 2 copper layers, 212.8 x 89.3 mm, 0 parts

Commit message: production files
Other:
- board text added: "screwhole m2.5 and led holes not aligned"
Changed lines of the file:
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@@
   (gr_line (start 91.425 48.275) (end 105.425 48.275) (layer "Edge.Cuts") (width 0.2))
   (gr_line (start 200.675 34.275) (end 186.675 34.275) (layer "Edge.Cuts") (width 0.2))
+  (gr_text "screwhole m2.5 and led holes not aligned\n" (at 132.207 23.876) (layer "F.Cu")
+    (effects (font (size 1.5 1.5) (thickness 0.3)))
+  )
   (gr_text "Didaktik 40\n" (at 193.04 189.611) (layer "F.Cu")
     (effects (font (size 1.5 1.5) (thickness 0.3)))
