File: Didaktik multilayout.kicad_sch (KiCad schematic)
At the start: 126 parts, among them J1 Conn_01x04_MountingPin, J2 AVR-ISP-6, J3 Conn_01x03, Q1 2N2222, SW1 SW_Push_45deg, SW10 SW_Push_45deg, SW11 SW_Push_45deg, SW12 SW_Push_45deg, SW13 SW_Push_45deg, SW14 SW_Push_45deg, SW15 SW_Push_45deg, SW16 SW_Push_45deg, SW17 SW_Push_45deg, SW18 SW_Push_45deg, SW19 SW_Push_45deg, SW2 SW_Push_45deg, SW20 SW_Push_45deg, SW21 SW_Push_45deg, SW22 SW_Push_45deg, SW23 SW_Push_45deg, SW24 SW_Push_45deg, SW25 SW_Push_45deg, SW26 SW_Push_45deg, SW27 SW_Push_45deg, SW28 SW_Push_45deg, SW29 SW_Push_45deg, SW3 SW_Push_45deg, SW30 SW_Push_45deg, SW31 SW_Push_45deg, SW31a1 SW_Push_45deg, SW32 SW_Push_45deg, SW32a1 SW_Push_45deg, SW33 SW_Push_45deg, SW33a1 SW_Push_45deg, SW34 SW_Push_45deg, SW34a1 SW_Push_45deg, SW34b1 SW_Push_45deg, SW35 SW_Push_45deg, SW35a1 SW_Push_45deg, SW35b1 SW_Push_45deg, SW35c1 SW_Push_45deg, SW36 SW_Push_45deg, SW36a1 SW_Push_45deg, SW36b1 SW_Push_45deg, SW36c1 SW_Push_45deg, SW37 SW_Push_45deg, SW37a1 SW_Push_45deg, SW37b1 SW_Push_45deg, SW38 SW_Push_45deg, SW38a1 SW_Push_45deg, SW39 SW_Push_45deg, SW39a1 SW_Push_45deg, SW4 SW_Push_45deg, SW40 SW_Push_45deg, SW40a1 SW_Push_45deg, SW41 RotaryEncoder_Switch, SW42 RotaryEncoder_Switch, SW5 SW_Push_45deg, SW6 SW_Push_45deg, SW7 SW_Push_45deg, SW8 SW_Push_45deg, SW9 SW_Push_45deg, U1 ATmega32U4-M, Y1 Crystal_GND24_Small

Commit message: changed sod123 to sod123f
Parts:
- D1, D10, D11, D12, D13, D14, D15, D16, D17, D18, D19, D2, D20, D21, D22, D23, D24, D26, D27, D28, D29, D3, D30, D31, D32, D33, D34, D35, D36, D37, D38, D39, D4, D40, D41, D5, D6, D7, D8, D9: footprint Diode_SMD:D_SOD-123 -> Diode_SMD:D_SOD-123F

Commit message: rgb pin changed from 42 to 1, new production files
Connections:
- net RGB: now also U1.1 (PE6); no longer U1.42 (AREF)
Changed lines of the file:
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@@
   (junction (at 195.58 123.19) (diameter 0) (color 0 0 0 0)
   )
-  (no_connect (at 68.58 87.63))
+  (no_connect (at 38.1 46.99))
   (wire (pts (xy 183.515 107.95) (xy 184.15 107.95))
     (stroke (width 0) (type default) (color 0 0 0 0))
@@
     )
   )
-  (global_label "RGB" (shape input) (at 38.1 46.99 180) (fields_autoplaced)
-    (effects (font (size 1.27 1.27)) (justify right))
-    (property "Intersheet References" "${INTERSHEET_REFS}" (id 0) (at -123.19 -0.635 0)
+  (global_label "RGB" (shape input) (at 68.58 87.63 0) (fields_autoplaced)
+    (effects (font (size 1.27 1.27)) (justify left))
+    (property "Intersheet References" "${INTERSHEET_REFS}" (id 0) (at 229.87 135.255 0)
       (effects (font (size 1.27 1.27)) hide)
     )

Commit message: V1.1
added double reset button, pinout
Parts:
- added SW_Reset2: SW_Push, Connector_PinHeader_2.54mm:PinHeader_1x02_P2.54mm_Vertical, symbol Switch:SW_Push
Connections:
- net GND: now also SW_Reset2.1
- net RESET: now also SW_Reset2.2
Changed lines of the file:
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@@
   (junction (at 215.9 67.31) (diameter 0) (color 0 0 0 0)
   )
+  (junction (at 121.92 186.055) (diameter 0) (color 0 0 0 0)
+  )
   (junction (at 220.98 41.275) (diameter 0) (color 0 0 0 0)
   )
@@
   (junction (at 195.58 83.185) (diameter 0) (color 0 0 0 0)
   )
+  (junction (at 111.76 186.055) (diameter 0) (color 0 0 0 0)
+  )
   (junction (at 165.1 88.265) (diameter 0) (color 0 0 0 0)
   )
@@
     (stroke (width 0) (type default) (color 0 0 0 0))
   )
+  (wire (pts (xy 121.92 186.055) (xy 121.92 188.595))
+    (stroke (width 0) (type default) (color 0 0 0 0))
+  )
   (wire (pts (xy 74.295 161.925) (xy 75.565 161.925))
     (stroke (width 0) (type default) (color 0 0 0 0))
@@
     (stroke (width 0) (type default) (color 0 0 0 0))
   )
+  (wire (pts (xy 111.76 186.055) (xy 111.76 188.595))
+    (stroke (width 0) (type default) (color 0 0 0 0))
+  )
   (wire (pts (xy 165.1 93.345) (xy 171.45 93.345))
     (stroke (width 0) (type default) (color 0 0 0 0))
@@
     (pin "2")
   )
+  (symbol (lib_id "Switch:SW_Push") (at 116.84 188.595 0) (unit 1)
+    (in_bom yes) (on_board yes)
+    (property "Reference" "SW_Reset2" (id 0) (at 116.84 193.04 0))
+    (property "Value" "SW_Push" (id 1) (at 116.84 190.5 0))
+    (property "Footprint" "Connector_PinHeader_2.54mm:PinHeader_1x02_P2.54mm_Vertical" (id 2) (at 116.84 183.515 0)
+      (effects (font (size 1.27 1.27)) hide)
+    )
+    (property "Datasheet" "~" (id 3) (at 116.84 183.515 0)
+      (effects (font (size 1.27 1.27)) hide)
+    )
+    (pin "1")
+    (pin "2")
+  )
   (symbol (lib_id "power:+5V") (at 111.76 131.445 0) (unit 1)
     (in_bom yes) (on_board yes) (fields_autoplaced)
@@
       (reference "SW_Reset1") (unit 1) (value "SW_Push") (footprint "random-keyboard-parts:SKQG-1155865")
     )
+    (path "/c419befe-d38d-4162-b568-009e5cc3779b"
+      (reference "SW_Reset2") (unit 1) (value "SW_Push") (footprint "Connector_PinHeader_2.54mm:PinHeader_1x02_P2.54mm_Vertical")
+    )
     (path "/12ccbf88-cdeb-48a3-a3a5-6440ea4100f4"
