File: Didaktik rp2040.kicad_pcb (KiCad board)
At the start: 2 copper layers, 209.6 x 76.2 mm, 143 parts, among them J1 Conn_01x04_MountingPin, J3 Conn_01x03, J5 SWD, Q1 2N2222, SW1 SW_Push_45deg, SW10 SW_Push_45deg, SW11 SW_Push_45deg, SW12 SW_Push_45deg, SW13 SW_Push_45deg, SW14 SW_Push_45deg, SW15 SW_Push_45deg, SW16 SW_Push_45deg, SW17 SW_Push_45deg, SW18 SW_Push_45deg, SW19 SW_Push_45deg, SW2 SW_Push_45deg, SW20 SW_Push_45deg, SW21 SW_Push_45deg, SW22 SW_Push_45deg, SW23 SW_Push_45deg, SW24 SW_Push_45deg, SW25 SW_Push_45deg, SW26 SW_Push_45deg, SW27 SW_Push_45deg, SW28 SW_Push_45deg, SW29 SW_Push_45deg, SW3 SW_Push_45deg, SW30 SW_Push_45deg, SW31 SW_Push_45deg, SW31a1 SW_Push_45deg, SW32 SW_Push_45deg, SW32a1 SW_Push_45deg, SW33 SW_Push_45deg, SW33a1 SW_Push_45deg, SW34 SW_Push_45deg, SW34a1 SW_Push_45deg, SW34b1 SW_Push_45deg, SW35 SW_Push_45deg, SW35a1 SW_Push_45deg, SW35b1 SW_Push_45deg, SW35c1 SW_Push_45deg, SW36 SW_Push_45deg, SW36a1 SW_Push_45deg, SW36b1 SW_Push_45deg, SW36c1 SW_Push_45deg, SW37 SW_Push_45deg, SW37a1 SW_Push_45deg, SW37b1 SW_Push_45deg, SW38 SW_Push_45deg, SW38a1 SW_Push_45deg, SW39 SW_Push_45deg, SW39a1 SW_Push_45deg, SW4 SW_Push_45deg, SW40 SW_Push_45deg, SW40a1 SW_Push_45deg, SW41 RotaryEncoder_Switch, SW42 RotaryEncoder_Switch, SW43 Reset, SW44 Boot, SW5 SW_Push_45deg, SW6 SW_Push_45deg, SW7 SW_Push_45deg, SW8 SW_Push_45deg, SW9 SW_Push_45deg, U1 XC6206PxxxMR, U2 RP2040, U3 W25Q128JVS, U4 USBLC6-2SC6, U5 74AHCT1G125, Y2 12MHz

Commit message: MCU routing on rp2040 version
Parts:
- moved U3 5.91 mm to (60.3, 52.7)
- moved C12 5.52 mm to (54.1, 50.3)
- moved R5 5.14 mm to (41.1, 90.5)
- moved C16 4.81 mm to (226.8, 50.0)
- moved C11 4.73 mm to (228.0, 50.0), turned to -90 degrees
- moved R12 4.50 mm to (232.2, 52.8)
- moved Q1 3.05 mm to (45.0, 85.7)
- moved C13 2.65 mm to (39.0, 63.8), turned to 180 degrees
- moved U4 2.27 mm to (228.6, 44.5)
- moved C6 2.22 mm to (232.1, 47.4)
- moved F1 2.19 mm to (231.8, 44.5)
- moved C17 1.79 mm to (39.0, 64.8), turned to 180 degrees
- moved C15 1.23 mm to (44.6, 76.8)
- moved C19 1.23 mm to (45.6, 76.8)
- moved U1 1.09 mm to (230.8, 50.4), turned to 0 degrees
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Routing:
- net +3V3: track 0.00 -> 262.4 mm, vias 0 -> 3
- net CS: track 0.00 -> 198.6 mm
- net D_P: track 0.00 -> 197.4 mm
- net D_N: track 0.00 -> 196.4 mm
- net SD1: track 0.00 -> 26.8 mm
- net SD2: track 0.00 -> 25.0 mm
- net SD3: track 0.00 -> 24.9 mm
- net GND: track 15.0 -> 38.5 mm, vias 10 -> 9
- net +1V1: track 0.00 -> 23.0 mm
- net QSPI_CLK: track 0.00 -> 22.0 mm
- net SD0: track 0.00 -> 21.7 mm
- net XTAL_IN: track 0.00 -> 15.5 mm
- net ROW0: track 400.0 -> 388.4 mm, vias 2 -> 1
- net /USB_BOOT: track 0.00 -> 8.38 mm
- net VBUS: track 247.2 -> 239.2 mm
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Other:
- board text added: "Didaktik 40 v2 by Calvin#0563"
- board text removed: "Didaktik 40 v1.1 by Calvin#0563"
