File: Didaktik rp2040.kicad_sch (KiCad schematic)
At the start: 32 parts, among them J1 Conn_01x04_MountingPin, J5 SWD, SW43 Reset, SW44 Boot, U1 XC6206PxxxMR, U2 RP2040, U3 W25Q128JVS, U4 USBLC6-2SC6, Y2 12MHz

Commit message: MCU routing on rp2040 version
Connections:
- net COL4: now also U2.14 (GPIO11)
- net ROW1: now also U2.2 (GPIO0)
Changed lines of the file:
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@@
     )
   )
-  (global_label "ROW1" (shape input) (at 196.215 57.15 0) (fields_autoplaced)
+  (global_label "ROW1" (shape input) (at 73.025 28.575 0) (fields_autoplaced)
     (effects (font (size 1.27 1.27)) (justify left))
-    (property "Intersheetrefs" "${INTERSHEET_REFS}" (at 203.8895 57.2294 0)
+    (property "Intersheetrefs" "${INTERSHEET_REFS}" (at 80.6995 28.6544 0)
       (effects (font (size 1.27 1.27)) (justify left) hide)
     )
@@
     )
   )
-  (global_label "COL4" (shape input) (at 195.58 85.725 0) (fields_autoplaced)
+  (global_label "COL4" (shape input) (at 73.025 56.515 0) (fields_autoplaced)
     (effects (font (size 1.27 1.27)) (justify left))
-    (property "Intersheetrefs" "${INTERSHEET_REFS}" (at 202.8312 85.6456 0)
+    (property "Intersheetrefs" "${INTERSHEET_REFS}" (at 80.2762 56.4356 0)
       (effects (font (size 1.27 1.27)) (justify left) hide)
     )
