File: Didaktik STEM.kicad_pcb (KiCad board)
At the start: 2 copper layers, 209.6 x 76.2 mm, 143 parts, among them J1 Conn_01x04_MountingPin, J3 Conn_01x03, J5 SWD, Q1 2N2222, SW1 SW_Push_45deg, SW10 SW_Push_45deg, SW11 SW_Push_45deg, SW12 SW_Push_45deg, SW13 SW_Push_45deg, SW14 SW_Push_45deg, SW15 SW_Push_45deg, SW16 SW_Push_45deg, SW17 SW_Push_45deg, SW18 SW_Push_45deg, SW19 SW_Push_45deg, SW2 SW_Push_45deg, SW20 SW_Push_45deg, SW21 SW_Push_45deg, SW22 SW_Push_45deg, SW23 SW_Push_45deg, SW24 SW_Push_45deg, SW25 SW_Push_45deg, SW26 SW_Push_45deg, SW27 SW_Push_45deg, SW28 SW_Push_45deg, SW29 SW_Push_45deg, SW3 SW_Push_45deg, SW30 SW_Push_45deg, SW31 SW_Push_45deg, SW31a1 SW_Push_45deg, SW32 SW_Push_45deg, SW32a1 SW_Push_45deg, SW33 SW_Push_45deg, SW33a1 SW_Push_45deg, SW34 SW_Push_45deg, SW34a1 SW_Push_45deg, SW34b1 SW_Push_45deg, SW35 SW_Push_45deg, SW35a1 SW_Push_45deg, SW35b1 SW_Push_45deg, SW35c1 SW_Push_45deg, SW36 SW_Push_45deg, SW36a1 SW_Push_45deg, SW36b1 SW_Push_45deg, SW36c1 SW_Push_45deg, SW37 SW_Push_45deg, SW37a1 SW_Push_45deg, SW37b1 SW_Push_45deg, SW38 SW_Push_45deg, SW38a1 SW_Push_45deg, SW39 SW_Push_45deg, SW39a1 SW_Push_45deg, SW4 SW_Push_45deg, SW40 SW_Push_45deg, SW40a1 SW_Push_45deg, SW41 RotaryEncoder_Switch, SW42 RotaryEncoder_Switch, SW43 Reset, SW44 Boot, SW5 SW_Push_45deg, SW6 SW_Push_45deg, SW7 SW_Push_45deg, SW8 SW_Push_45deg, SW9 SW_Push_45deg, U1 XC6206PxxxMR, U2 RP2040, U3 W25Q128JVS, U4 USBLC6-2SC6, U5 74AHCT1G125, Y2 12MHz

Commit message: added STEM project WIP
Parts:
- removed C10: 22pF, Capacitor_SMD:C_0402_1005Metric
- removed C11, C13, C17: 1uF, Capacitor_SMD:C_0402_1005Metric
- removed C12, C14, C15, C18, C19, C20, C21, C22, C23, C24: 100nF, Capacitor_SMD:C_0402_1005Metric
- removed C16: 10uF, Capacitor_SMD:C_0402_1005Metric
- removed J5: SWD, Connector_PinSocket_2.54mm:PinSocket_1x05_P2.54mm_Vertical
- removed R10: 27R, Resistor_SMD:R_0402_1005Metric
- removed R11, R12: 1k, Resistor_SMD:R_0402_1005Metric
- removed SW44: Boot, Keebio-Parts:SW_SPST_TL3342
- removed U1: XC6206PxxxMR, Package_TO_SOT_SMD:SOT-23
- removed U2: RP2040, Sleep-lib:RP2040-QFN-56
- removed U3: W25Q128JVS, Package_SO:SOIC-8_5.23x5.23mm_P1.27mm
- removed U4: USBLC6-2SC6, Package_TO_SOT_SMD:SOT-23-6
- removed Y2: 12MHz, Crystal:Crystal_SMD_3225-4Pin_3.2x2.5mm
- added C2: 1uF, Capacitor_SMD:C_0603_1608Metric, B.Cu at (232.6, 47.5)
- added C25: 100nF, Capacitor_SMD:C_0603_1608Metric, B.Cu at (25.4, 61.2)
- added C26: 100nF, Capacitor_SMD:C_0603_1608Metric, B.Cu at (25.4, 63.8)
- added C27: 100nF, Capacitor_SMD:C_0603_1608Metric, B.Cu at (21.4, 53.7)
- added C3: 1uF, Capacitor_SMD:C_0603_1608Metric, B.Cu at (227.6, 49.8)
- added C4: 4.7uF, Capacitor_SMD:C_0603_1608Metric, B.Cu at (29.4, 58.7)
- added C5: 1uF, Capacitor_SMD:C_0603_1608Metric, B.Cu at (29.4, 61.2)
- added C7: 100nF, Capacitor_SMD:C_0603_1608Metric, B.Cu at (25.4, 53.7)
- added C8: 100nF, Capacitor_SMD:C_0603_1608Metric, B.Cu at (25.4, 56.2)
- added Q2: 2N7002, Package_TO_SOT_SMD:SOT-23, B.Cu at (35.1, 79.3)
- added R3: 10k, Resistor_SMD:R_0603_1608Metric, B.Cu at (31.0, 74.6)
- added U6: USBLC6-2SC6, Package_TO_SOT_SMD:SOT-23-6, B.Cu at (228.6, 44.5)
- added U7: STM32F072C8Tx, Package_QFP:LQFP-48_7x7mm_P0.5mm, B.Cu at (49.2, 70.6)
- added U8: XC6206PxxxMR-Regulator_Linear, Package_TO_SOT_SMD:SOT-23, B.Cu at (230.4, 50.0)
- C6: value 1uF -> 4.7u; footprint Capacitor_SMD:C_0402_1005Metric -> Capacitor_SMD:C_0603_1608Metric
- C9: value 22pF -> 1u; footprint Capacitor_SMD:C_0402_1005Metric -> Capacitor_SMD:C_0603_1608Metric
- R1: value 1k -> 10k; footprint Resistor_SMD:R_0402_1005Metric -> Resistor_SMD:R_0603_1608Metric
- R2, R4, R6: footprint Resistor_SMD:R_0402_1005Metric -> Resistor_SMD:R_0603_1608Metric
- R7: value 27R -> 100k; footprint Resistor_SMD:R_0402_1005Metric -> Resistor_SMD:R_0603_1608Metric
- SW43: value Reset -> RST; footprint Keebio-Parts:SW_SPST_TL3342 -> Button_Switch_SMD:SW_SPST_SKQG_WithoutStem
- moved C6 203.4 mm to (29.4, 63.8), turned to 180 degrees
- moved C9 36.0 mm to (25.4, 58.7), turned to 180 degrees
- moved R7 19.0 mm to (31.0, 77.1), turned to 180 degrees
- moved R1 18.7 mm to (31.0, 72.1), turned to 180 degrees
- moved SW43 16.7 mm to (35.7, 72.2)
Connections:
- C6 pad 1: +5V -> BOOT0
- C6 pad 2: GND -> Net-(Q2-G)
- C9 pad 2: XTAL_IN -> NRST
- R1 pad 1: /XTAL_O -> +3V3
- R1 pad 2: XTAL_OUT -> NRST
- R7 pad 1: D_P -> Net-(Q2-G)
- R7 pad 2: /D_+ -> GND
- SW43 pad 1: RESET -> BOOT0
- SW43 pad 2: GND -> +3V3
Routing:
- net +3V3: track 266.4 -> 11.2 mm, vias 3 -> 0
- net CS: track 199.9 -> 0.00 mm
- net D_P: track 199.9 -> 0.00 mm
- net D_N: track 198.6 -> 0.00 mm
- net SD1: track 27.4 -> 0.00 mm
- net SD2: track 26.0 -> 0.00 mm
- net +1V1: track 23.0 -> 0.00 mm
- net SD0: track 21.7 -> 0.00 mm
- net SD3: track 21.1 -> 0.00 mm
- net GND: track 38.5 -> 18.3 mm, vias 10 -> 8
- net QSPI_CLK: track 20.1 -> 0.00 mm
- net XTAL_IN: track 15.5 -> 0.00 mm
- net /USB_BOOT: track 8.38 -> 0.00 mm
- net XTAL_OUT: track 6.46 -> 0.00 mm
- net (no net): track 0.00 -> 6.30 mm
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- removed copper zone on B.Cu, net +1V1
- removed copper zone on B.Cu, net +3V3
