File: Project/Didaktik switchplate.kicad_pcb (KiCad board)
At the start: 2 copper layers, 209.6 x 85.9 mm, 0 parts

Commit message: update
Parts:
- added REF**: MountingHole_2.2mm_M2, MountingHole:MountingHole_2.2mm_M2, F.Cu at (231.8, 110.1)
- added REF**: MountingHole_2.2mm_M2, MountingHole:MountingHole_2.2mm_M2, F.Cu at (231.8, 29.5)
- added REF**: MountingHole_2.2mm_M2, MountingHole:MountingHole_2.2mm_M2, F.Cu at (41.3, 110.2)
- added REF**: MountingHole_2.2mm_M2, MountingHole:MountingHole_2.2mm_M2, F.Cu at (41.3, 29.5)
Other:
- outline, holes or cut-outs redrawn
