File: Project/components.kicad_sch (KiCad schematic)
At the start: 11 parts, among them J3 Conn_01x03, Q1 2N2222, U5 74AHCT1G125

Commit message: added STM project
Parts:
- renumbered C1 to C10, D43 to D?, D42 to D?, J3 to J?, LS1 to LS?, Q1 to Q?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
