File: Project/matrix.kicad_sch (KiCad schematic)
At the start: 98 parts, among them SW1 SW_Push_45deg, SW10 SW_Push_45deg, SW11 SW_Push_45deg, SW12 SW_Push_45deg, SW13 SW_Push_45deg, SW14 SW_Push_45deg, SW15 SW_Push_45deg, SW16 SW_Push_45deg, SW17 SW_Push_45deg, SW18 SW_Push_45deg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

Commit message: added STM project
Parts:
- renumbered D12 to D?, D35 to D?, D9 to D?, D11 to D?, D13 to D?, D14 to D?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
